File: stepdown24v_to_5v_1A/WBDesign4_CadSoftEAGLE/ExportFiles/Schematic/webench_schematic_exchange_design_6559895_4_Eagle/Eagle/2021-02-22_22-45-18/2021-02-22_22-45-18.sch (EAGLE design)
At the start: 14 parts

Commit message: BOM for stepdown
Parts:
- added R1: 10k, Components:RESISTOR-0603
- added R2: 1k, Components:RESISTOR-0603
- RFBT: value 111k -> 100k
Connections:
- new net N$1: CIN.2, J1.1, LMR14010ADDC.VIN@5, SV1.3, TP1.TP
- new net N$4: R1.2, RFBT.1
- new net N$5: R1.1, R2.2
- net 2: now also R2.1; no longer RFBT.1
- net GND: no longer CIN.2, J1.1, LMR14010ADDC.VIN@5, SV1.3, TP1.TP
Other:
- moved on the sheet: RFBT
Changed lines of the file:
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@@
 <part name="COUT_2" library="Components" deviceset="CAPACITOR" device="-0603" value="10uF"/>
 <part name="COUT" library="Components" deviceset="CAPACITOR" device="-0603" value="10uF"/>
-<part name="RFBT" library="Components" deviceset="RESISTOR" device="-0603" value="111k"/>
+<part name="RFBT" library="Components" deviceset="RESISTOR" device="-0603" value="100k"/>
 <part name="RFBB" library="Components" deviceset="RESISTOR" device="-0603" value="20k"/>
 <part name="D1" library="Components" deviceset="DIODE" device="-DFN0603-2" value="550mV"/>
@@
 <part name="SUPPLY5" library="supply2" library_urn="urn:adsk.eagle:library:372" deviceset="GND" device=""/>
 <part name="SUPPLY6" library="supply2" library_urn="urn:adsk.eagle:library:372" deviceset="GND" device=""/>
+<part name="R1" library="Components" deviceset="RESISTOR" device="-0603" value="10k"/>
+<part name="R2" library="Components" deviceset="RESISTOR" device="-0603" value="1k"/>
 </parts>
 <sheets>
@@
 <attribute name="VALUE" x="232.664" y="60.96" size="1.778" layer="96" align="top-left"/>
 </instance>
-<instance part="RFBT" gate="G$1" x="204.47" y="74.676" smashed="yes" rot="R90">
-<attribute name="NAME" x="208.0514" y="75.946" size="1.778" layer="95"/>
-<attribute name="VALUE" x="207.772" y="73.406" size="1.778" layer="96"/>
+<instance part="RFBT" gate="G$1" x="204.47" y="79.756" smashed="yes" rot="R90">
+<attribute name="NAME" x="208.0514" y="81.026" size="1.778" layer="95"/>
+<attribute name="VALUE" x="207.772" y="78.486" size="1.778" layer="96"/>
 </instance>
 <instance part="RFBB" gate="G$1" x="204.47" y="42.164" smashed="yes" rot="R90">
@@
 <instance part="SUPPLY6" gate="GND" x="133.604" y="27.94" smashed="yes">
 <attribute name="VALUE" x="131.699" y="24.765" size="1.778" layer="96"/>
+</instance>
+<instance part="R1" gate="G$1" x="204.47" y="69.596" smashed="yes" rot="R90">
+<attribute name="NAME" x="207.0354" y="70.358" size="1.778" layer="95"/>
+<attribute name="VALUE" x="206.756" y="67.818" size="1.778" layer="96"/>
+</instance>
+<instance part="R2" gate="G$1" x="204.47" y="59.436" smashed="yes" rot="R90">
+<attribute name="NAME" x="206.7814" y="59.944" size="1.778" layer="95"/>
+<attribute name="VALUE" x="206.502" y="57.404" size="1.778" layer="96"/>
 </instance>
 </instances>
@@
 <pinref part="RFBB" gate="G$1" pin="2"/>
 <wire x1="204.47" y1="47.244" x2="204.47" y2="49.784" width="0.1524" layer="91"/>
-<wire x1="204.47" y1="66.04" x2="204.47" y2="49.53" width="0" layer="91"/>
-<pinref part="RFBT" gate="G$1" pin="1"/>
-<wire x1="204.47" y1="69.596" x2="204.47" y2="49.53" width="0.1524" layer="91"/>
+<pinref part="R2" gate="G$1" pin="1"/>
+<wire x1="204.47" y1="54.356" x2="204.47" y2="49.784" width="0.1524" layer="91"/>
+<junction x="204.47" y="49.784"/>
 </segment>
 <segment>
@@
 <segment>
 <pinref part="RFBT" gate="G$1" pin="2"/>
-<wire x1="204.47" y1="79.756" x2="204.47" y2="86.36" width="0.1524" layer="91"/>
+<wire x1="204.47" y1="84.836" x2="204.47" y2="86.36" width="0.1524" layer="91"/>
 </segment>
 <segment>
@@
 <wire x1="247.65" y1="50.8" x2="229.87" y2="50.8" width="0.1524" layer="91"/>
 <pinref part="IOUT" gate="1" pin="-@2"/>
-<wire x1="29.21" y1="30.48" x2="54.61" y2="30.48" width="0" layer="91"/>
 <wire x1="54.61" y1="30.48" x2="133.604" y2="30.48" width="0" layer="91"/>
 <wire x1="133.604" y1="30.48" x2="229.87" y2="30.48" width="0" layer="91"/>
 <wire x1="229.87" y1="30.48" x2="278.13" y2="30.48" width="0" layer="91"/>
 <wire x1="278.13" y1="30.48" x2="278.13" y2="43.18" width="0" layer="91"/>
-<wire x1="29.21" y1="58.166" x2="29.21" y2="58.42" width="0" layer="91"/>
+<pinref part="CIN" gate="G$1" pin="1"/>
+<wire x1="54.61" y1="60.96" x2="54.61" y2="30.48" width="0.1524" layer="91"/>
+<wire x1="229.87" y1="50.8" x2="229.87" y2="30.48" width="0.1524" layer="91"/>
+<junction x="229.87" y="50.8"/>
+<junction x="229.87" y="30.48"/>
+<pinref part="SUPPLY6" gate="GND" pin="GND"/>
+<junction x="133.604" y="30.48"/>
+</segment>
+</net>
+<net name="N$2" class="0">
+<segment>
+<wire x1="113.03" y1="86.36" x2="166.37" y2="86.36" width="0" layer="91"/>
+<pinref part="L2" gate="G$1" pin="1"/>
+<wire x1="167.64" y1="86.36" x2="113.03" y2="86.36" width="0.1524" layer="91"/>
+<pinref part="LMR14010ADDC" gate="1" pin="SW@6"/>
+<junction x="113.03" y="86.36"/>
+</segment>
+</net>
+<net name="N$1" class="0">
+<segment>
 <pinref part="TP1" gate="G$1" pin="TP"/>
 <wire x1="35.56" y1="116.84" x2="35.56" y2="114.3" width="0.1524" layer="91"/>
@@
 <wire x1="54.61" y1="93.98" x2="35.56" y2="93.98" width="0.1524" layer="91"/>
 <pinref part="SV1" gate="G$1" pin="3"/>
-<wire x1="0" y1="93.98" x2="29.21" y2="93.98" width="0.1524" layer="91"/>
-<wire x1="29.21" y1="93.98" x2="35.56" y2="93.98" width="0.1524" layer="91"/>
-<junction x="29.21" y="93.98"/>
-<wire x1="29.21" y1="93.98" x2="29.21" y2="58.166" width="0.1524" layer="91"/>
-<wire x1="29.21" y1="58.166" x2="29.21" y2="30.48" width="0.1524" layer="91"/>
-<junction x="29.21" y="58.166"/>
-<pinref part="CIN" gate="G$1" pin="1"/>
-<wire x1="54.61" y1="60.96" x2="54.61" y2="30.48" width="0.1524" layer="91"/>
-<junction x="54.61" y="30.48"/>
-<wire x1="229.87" y1="50.8" x2="229.87" y2="30.48" width="0.1524" layer="91"/>
-<junction x="229.87" y="50.8"/>
-<junction x="229.87" y="30.48"/>
-<pinref part="SUPPLY6" gate="GND" pin="GND"/>
-<junction x="133.604" y="30.48"/>
-</segment>
-</net>
-<net name="N$2" class="0">
-<segment>
-<wire x1="113.03" y1="86.36" x2="166.37" y2="86.36" width="0" layer="91"/>
-<pinref part="L2" gate="G$1" pin="1"/>
-<wire x1="167.64" y1="86.36" x2="113.03" y2="86.36" width="0.1524" layer="91"/>
-<pinref part="LMR14010ADDC" gate="1" pin="SW@6"/>
-<junction x="113.03" y="86.36"/>
-</segment>
-</net>
+<wire x1="0" y1="93.98" x2="35.56" y2="93.98" width="0.1524" layer="91"/>
+</segment>
+</net>
+<net name="N$3" class="0">
+<segment>
+<wire x1="29.21" y1="58.166" x2="29.21" y2="58.42" width="0" layer="91"/>
+</segment>
+</net>
+<net name="N$4" class="0">
+<segment>
+<pinref part="RFBT" gate="G$1" pin="1"/>
+<pinref part="R1" gate="G$1" pin="2"/>
+</segment>
+</net>
+<net name="N$5" class="0">
+<segment>
+<pinref part="R1" gate="G$1" pin="1"/>
+<pinref part="R2" gate="G$1" pin="2"/>
+</segment>
+</net>
